File: hw/picobaloon/picobaloon.kicad_pcb (KiCad board)
At the start: 2 copper layers, 41 x 56.3 mm, 45 parts, among them J1 SOLAR+, J2 SWD, J3 DEBUG, J4 GPS_ANT, J5 ANT, J6 SOLAR-, Q1 BC847, Q2 BC857, U1 LMT87DCK, U2 MCP1640CH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

Commit message: HW revision 2 - added pressure sensor
Parts:
- added C16: 100n, Capacitor_SMD:C_0805_2012Metric, F.Cu at (225.6, 132.1)
- added R12: 10k, Resistor_SMD:R_0805_2012Metric, F.Cu at (221.6, 128.7)
- added R13: 10k, Resistor_SMD:R_0805_2012Metric, F.Cu at (221.6, 130.7)
- added U6: MS5607-02BA, Package_LGA:LGA-8_3x5mm_P1.25mm, F.Cu at (226.2, 129.4)
- J2: footprint Connector_PinHeader_2.54mm:PinHeader_1x05_P2.54mm_Vertical -> Connector_PinHeader_2.54mm:PinHeader_1x04_P2.54mm_Vertical
- moved J2 0.16 mm to (223.3, 120.2), turned to 270 degrees
Connections:
- U3 pad 26: (no net) -> /SCL
- U3 pad 27: (no net) -> /SDA
Routing:
- net GND: track 233.7 -> 257.0 mm
- net /SDA: track 0.00 -> 14.8 mm
- net +3V3: track 216.9 -> 230.7 mm
- net /SCL: track 0.00 -> 8.84 mm
- net /SWDIO: track 9.65 -> 17.2 mm
- net /SWCLK: track 10.9 -> 13.8 mm
- net /DIO0: track 49.5 -> 48.8 mm
Other:
- board text added: "Brno 03/2019"
- board text added: "Czech Republic"
- board text removed: "PicoBalloon Czech Republic Brno, March 2019"

Commit message: HW revision 3. Added resistors for simple esd protection
Parts:
- added R14: 1M, Resistor_SMD:R_0805_2012Metric, F.Cu at (229.5, 145.1)
- added R15: 1M, Resistor_SMD:R_0805_2012Metric, F.Cu at (233.8, 114.9)
- C2: value CP -> 3F/3V
- moved C12 2.80 mm to (228.0, 95.2)
- moved C13 2.03 mm to (228.0, 93.3), turned to 0 degrees
Routing:
- net GND: track 257.0 -> 264.4 mm
- net Net-(J4-Pad1): track 6.85 -> 10.6 mm
- net +3V3: track 230.7 -> 228.1 mm
- net Net-(J5-Pad1): track 4.57 -> 7.03 mm
Other:
- board text added: "Czech Republic Brno 03/2019"
- board text removed: "Brno 03/2019"
- board text removed: "Czech Republic"

Commit message: Updated schematic to match the final symbol in the official repo
Parts:
- C2: value 3F/3V -> 3F3/3V
Changed lines of the file:
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@@
   )
   (setup
-    (last_trace_width 0.8)
+    (last_trace_width 0.25)
     (user_trace_width 0.3)
     (user_trace_width 0.4)
@@
       (effects (font (size 1 1) (thickness 0.15)) (justify mirror))
     )
-    (fp_text value 3F/3V (at 1.75 -5.25) (layer B.Fab)
+    (fp_text value 3F3/3V (at 1.75 -5.25) (layer B.Fab)
       (effects (font (size 1 1) (thickness 0.15)) (justify mirror))
     )
